File: PCB/biky.kicad_pcb (KiCad board)
At the start: 2 copper layers, 124.7 x 34.5 mm, 51 parts, among them J1 Conn_02x05_Odd_Even, Q1 PN2222A, Q2 PN2222A, Q3 PN2222A, Q4 MPSA42

Commit message: no regulator
Parts:
- removed D24: Vz10V, Diode_THT:D_DO-35_SOD27_P12.70mm_Horizontal
- removed Q4: MPSA42, Package_TO_SOT_THT:TO-92_Inline
- removed R15, R16, R17: 1k, Resistor_THT:R_Axial_DIN0207_L6.3mm_D2.5mm_P10.16mm_Horizontal
- moved R18 32.9 mm to (150.2, 101.5)
- moved D20 23.7 mm to (184.5, 81.5)
- moved D22 8.00 mm to (194.7, 84.7), turned to 180 degrees
- moved J1 5.18 mm to (201.0, 80.5)
- moved D21 4.48 mm to (190.5, 95.7)
- moved D25 1.48 mm to (205.7, 93.2)
- moved R1 1.27 mm to (115.5, 93.8)
- moved D23 1.21 mm to (200.7, 92.5)
- moved C1 0.29 mm to (172.7, 88.7)
Connections:
- A1 pad 17: +3V3 -> Net-(A1-Pad17)
- C1 pad 1: VDD -> +5V
- D13 pad 2: +3V3 -> +5V
- D14 pad 2: +3V3 -> +5V
- D15 pad 2: +3V3 -> +5V
- D16 pad 2: +3V3 -> +5V
- D17 pad 2: +3V3 -> +5V
- D18 pad 2: +3V3 -> +5V
- D19 pad 2: +3V3 -> +5V
- D20 pad 1: Net-(D20-Pad1) -> +5V
- D21 pad 1: /Dynamo+ -> +5V
- D21 pad 2: GND -> /Dynamo-
- D22 pad 1: Net-(D20-Pad1) -> /Dynamo+
- D22 pad 2: /Dynamo- -> GND
- J1 pad 4: +3V3 -> +5V
Routing:
- net +5V: track 0.00 -> 182.2 mm
- net +3V3: track 145.3 -> 0.00 mm
- net VDD: track 57.5 -> 0.00 mm
- net /LightButtonLeft: track 14.2 -> 51.8 mm
- net Net-(D1-Pad2): track 112.7 -> 79.0 mm
- net Net-(D20-Pad1): track 32.4 -> 0.00 mm
- net GND: track 183.3 -> 160.0 mm
- net /LightButtonRigh: track 67.6 -> 90.8 mm
- net /Dynamo+: track 29.8 -> 10.0 mm
- net Net-(Q4-Pad2): track 15.7 -> 0.00 mm
- net Net-(D16-Pad1): track 85.9 -> 95.8 mm
- net Net-(D24-Pad1): track 9.35 -> 0.00 mm
- net /Leftswitch: track 118.7 -> 127.1 mm, vias 1 -> 0
- net /Segment1: track 41.7 -> 34.7 mm
- net Net-(D13-Pad1): track 131.8 -> 137.1 mm
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